File: ControllerPCB/ControllerPCB.kicad_sch (KiCad schematic)
At the start: 43 parts, among them J1 USB_B_Micro, J2 A-DF 09 A/KG-T4S, J3 Screw_Terminal_01x02, J4 MotorDriverSocket, J5 UISocket, J6 Pi JST, J7 Conn_02x02_Row_Letter_First, SW1 SW_Push_Dual_x2, SW2 SW_Push_Dual_x2, U1 AMS1117-3.3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

Commit message: Rev 2 of controller PCB
Parts:
- removed R7, R8: 10k, Resistor_SMD:R_0805_2012Metric_Pad1.20x1.40mm_HandSolder, symbol Device:R
- added D6: WS2812B, LED_SMD:LED_WS2812B_PLCC4_5.0x5.0mm_P3.2mm, symbol LED:WS2812B
- added D7, D8: LED, LED_SMD:LED_0805_2012Metric_Pad1.15x1.40mm_HandSolder, symbol Device:LED
- added R10, R11: 10k, Resistor_SMD:R_0805_2012Metric_Pad1.20x1.40mm_HandSolder, symbol Device:R
- added TP4, TP5, TP6, TP7, TP8, TP9: TestPoint, TestPoint:TestPoint_Pad_1.5x1.5mm, symbol Connector:TestPoint
- R3, R4: value 10k -> 5.1k
Connections:
- net +3.3V: now also R10.2, R11.2
- net +5V: now also J6.1 (Pin_1), D6.1 (VDD); no longer J6.4 (Pin_4)
- net GND: now also J6.2 (Pin_2), D6.3 (VSS); no longer J6.5 (Pin_5)
- net at U2.11 (IO18): now also J6.5 (Pin_5); no longer J6.3 (Pin_3)
- net at U2.19 (IO11): now also J6.3 (Pin_3); no longer J6.1 (Pin_1)
- net at U2.21 (IO13): now also J6.4 (Pin_4); no longer J6.2 (Pin_2)
- net at U2.24 (IO47): now also TP8.1; no longer J5.8 (Pin_8)
- net at U2.25 (IO48): now also TP9.1; no longer J5.9 (Pin_9)
- net at C2.2, U2.27 (IO0): now also J5.8 (Pin_8), SW2.3 (D), R11.1; no longer SW2.2 (D)
- net at C1.2, U2.3 (EN): now also J5.9 (Pin_9), SW1.3 (D), R10.1; no longer SW1.2 (D)
- net at U2.32 (MTCK/IO39): now also TP4.1
- net at U2.33 (MTDO/IO40): now also TP5.1
- net at U2.34 (MTDI/IO41): now also TP6.1
- net at U2.35 (MTMS/IO42): now also TP7.1
- net at J2.1, U2.8 (IO15): now also D8.1 (K); no longer R3.2
- net at J2.3, U2.9 (IO16): now also D7.1 (K); no longer R4.2
- net at J5.10 (Pin_10): now also D6.2 (DOUT); no longer U6.13 (B1)
- new net: D7.2 (A), R4.2
- new net: D8.2 (A), R3.2
- new net: D6.4 (DIN), U6.13 (B1)
Other:
- moved on the sheet: D3, D4, J1, J6, R3, R4, U5
